Commit message: fix naming

File: robots/nexus_base.urdf.xacro (robot description, xacro)
@@ -10,11 +10,11 @@
   <!-- The following xacro:included files set up definitions of parts of the robot body -->
   <!-- misc common stuff? -->
-  <xacro:include filename="$(find nexus_robot)/urdf/common.xacro" />
+  <xacro:include filename="$(find nexus_widowx_gazebo)/urdf/common.xacro" />
   <!-- nexus base -->
-  <xacro:include filename="$(find nexus_robot)/urdf/nexus_base/base.urdf.xacro" />
+  <xacro:include filename="$(find nexus_widowx_gazebo)/urdf/nexus_base/base.urdf.xacro" />
   <!-- controller manager -->
-  <xacro:include filename="$(find nexus_robot)/controller/ros_controller.urdf.xacro" />
+  <xacro:include filename="$(find nexus_widowx_gazebo)/controller/ros_controller.urdf.xacro" />
   <!-- materials for visualization -->
-  <xacro:include filename="$(find nexus_robot)/urdf/materials.urdf.xacro" />
+  <xacro:include filename="$(find nexus_widowx_gazebo)/urdf/materials.urdf.xacro" />
   <!-- The first use of a macro.  This one was defined in base.urdf.xacro above.
        A macro like this will expand to a set of link and joint definitions, and to additional

File: robots/nexus_base_arm.urdf.xacro (robot description, xacro)
@@ -9,15 +9,15 @@
        name="nexus_base_arm" >
   <!-- misc common stuff? -->
-  <xacro:include filename="$(find nexus_robot)/urdf/common.xacro" />
+  <xacro:include filename="$(find nexus_widowx_gazebo)/urdf/common.xacro" />
   <!-- nexus base -->
-  <xacro:include filename="$(find nexus_robot)/urdf/nexus_base/base.urdf.xacro" />
+  <xacro:include filename="$(find nexus_widowx_gazebo)/urdf/nexus_base/base.urdf.xacro" />
   <!-- widowx arm -->
-  <xacro:include filename="$(find nexus_robot)/urdf/widowx_arm/common_colours.xacro" />
-  <xacro:include filename="$(find nexus_robot)/urdf/widowx_arm/common_materials.xacro" />
-  <xacro:include filename="$(find nexus_robot)/urdf/widowx_arm/widowx.urdf.xacro" />
+  <xacro:include filename="$(find nexus_widowx_gazebo)/urdf/widowx_arm/common_colours.xacro" />
+  <xacro:include filename="$(find nexus_widowx_gazebo)/urdf/widowx_arm/common_materials.xacro" />
+  <xacro:include filename="$(find nexus_widowx_gazebo)/urdf/widowx_arm/widowx.urdf.xacro" />
   <!-- controller manager -->
-  <xacro:include filename="$(find nexus_robot)/controller/ros_controller.urdf.xacro" />
+  <xacro:include filename="$(find nexus_widowx_gazebo)/controller/ros_controller.urdf.xacro" />
   <!-- materials for visualization -->
-  <xacro:include filename="$(find nexus_robot)/urdf/materials.urdf.xacro" />
+  <xacro:include filename="$(find nexus_widowx_gazebo)/urdf/materials.urdf.xacro" />
   <!-- The first use of a macro.  This one was defined in base.urdf.xacro above.
        A macro like this will expand to a set of link and joint definitions, and to additional

File: urdf/nexus_base/base.urdf.xacro (robot description, xacro)
@@ -8,6 +8,6 @@
        xmlns:xacro="http://ros.org/wiki/xacro">
   <!-- sensors -->
-  <xacro:include filename="$(find nexus_robot)/urdf/nexus_base/base.gazebo.xacro"/>
-  <xacro:include filename="$(find nexus_robot)/urdf/nexus_base/base.transmission.xacro"/>
+  <xacro:include filename="$(find nexus_widowx_gazebo)/urdf/nexus_base/base.gazebo.xacro"/>
+  <xacro:include filename="$(find nexus_widowx_gazebo)/urdf/nexus_base/base.transmission.xacro"/>
   <!-- simplified box collision geometry for base -->
   <xacro:property name="base_size_x" value="0.380"/>
@@ -104,5 +104,5 @@
         <origin xyz="0 0 0.02" rpy="0 0 0"/>
         <geometry>
-          <mesh filename="package://nexus_robot/meshes/mecanum_wheel.dae">
+          <mesh filename="package://nexus_widowx_gazebo/meshes/mecanum_wheel.dae">
             <scale>${caster_scale} ${caster_scale} ${caster_scale}</scale>
           </mesh>
@@ -151,5 +151,5 @@
         <origin xyz="0 0 0.02" rpy="0 0 0"/>
         <geometry>
-          <mesh filename="package://nexus_robot/meshes/mecanum_wheel.dae" />
+          <mesh filename="package://nexus_widowx_gazebo/meshes/mecanum_wheel.dae" />
           <scale>${caster_scale} ${caster_scale} ${caster_scale}</scale>
         </geometry>
@@ -198,5 +198,5 @@
         <origin xyz="0 0 0.02" rpy="0 0 0"/>
         <geometry>
-          <mesh filename="package://nexus_robot/meshes/mecanum_wheel.dae" />
+          <mesh filename="package://nexus_widowx_gazebo/meshes/mecanum_wheel.dae" />
           <scale>${caster_scale} ${caster_scale} ${caster_scale}</scale>
         </geometry>
@@ -244,5 +244,5 @@
         <origin xyz="0 0 0.02" rpy="0 0 0"/>
         <geometry>
-          <mesh filename="package://nexus_robot/meshes/mecanum_wheel.dae" />
+          <mesh filename="package://nexus_widowx_gazebo/meshes/mecanum_wheel.dae" />
           <scale>${caster_scale} ${caster_scale} ${caster_scale}</scale>
         </geometry>

File: urdf/widowx_arm/common_materials.xacro (robot description, xacro)
@@ -1,5 +1,5 @@
 <?xml version="1.0"?>
 <robot xmlns:xacro="http://ros.org/wiki/xacro">
-	<xacro:include filename="$(find nexus_robot)/urdf/widowx_arm/common_colours.xacro"/>
+	<xacro:include filename="$(find nexus_widowx_gazebo)/urdf/widowx_arm/common_colours.xacro"/>
 	<xacro:macro name="material_yellow">
 		<material name="">

File: urdf/widowx_arm/widowx.urdf.xacro (robot description, xacro)
@@ -3,6 +3,6 @@
    <property name="M_SCALE" value="0.001"/>
    <property name="M_PI" value="3.14159"/>
-   <xacro:include filename="$(find nexus_robot)/urdf/widowx_arm/common_materials.xacro" />
-   <xacro:include filename="$(find nexus_robot)/urdf/widowx_arm/widowx.transmission.xacro" />
+   <xacro:include filename="$(find nexus_widowx_gazebo)/urdf/widowx_arm/common_materials.xacro" />
+   <xacro:include filename="$(find nexus_widowx_gazebo)/urdf/widowx_arm/widowx.transmission.xacro" />
    <xacro:macro name="default_inertia">
       <inertia ixx="0.002" ixy="0.0" ixz="0.0" iyy="0.002" iyz="0.0" izz="0.002" />
@@ -21,5 +21,5 @@
             <origin xyz="0 0 0" rpy="0 0 0" />
             <geometry>
-               <mesh filename="package://nexus_robot/meshes/base_link.stl"/>
+               <mesh filename="package://nexus_widowx_gazebo/meshes/base_link.stl"/>
             </geometry>
             <xacro:material_black />
@@ -28,5 +28,5 @@
             <origin xyz="0 0 0" rpy="0 0 0" />
             <geometry>
-               <mesh filename="package://nexus_robot/meshes/base_link.stl"/>
+               <mesh filename="package://nexus_widowx_gazebo/meshes/base_link.stl"/>
             </geometry>
          </collision>
@@ -41,12 +41,12 @@
             <origin xyz="0 0 0" rpy="0 0 0" />
             <geometry>
-               <mesh filename="package://nexus_robot/meshes/shoulder_link.stl" />
-            </geometry>
-            <xacro:material_black />
-         </visual>
-         <collision>
-            <origin xyz="0 0 0" rpy="0 0 0" />
-            <geometry>
-               <mesh filename="package://nexus_robot/meshes/shoulder_link.stl"/>
+               <mesh filename="package://nexus_widowx_gazebo/meshes/shoulder_link.stl" />
+            </geometry>
+            <xacro:material_black />
+         </visual>
+         <collision>
+            <origin xyz="0 0 0" rpy="0 0 0" />
+            <geometry>
+               <mesh filename="package://nexus_widowx_gazebo/meshes/shoulder_link.stl"/>
             </geometry>
          </collision>
@@ -62,12 +62,12 @@
             <!--origin xyz="0 0 0" rpy="0 0 0" /-->
             <geometry>
-               <mesh filename="package://nexus_robot/meshes/biceps_link.stl" />
-            </geometry>
-            <xacro:material_black />
-         </visual>
-         <collision>
-            <origin xyz="0 0 0" rpy="0 0 0" />
-            <geometry>
-               <mesh filename="package://nexus_robot/meshes/biceps_link.stl" />
+               <mesh filename="package://nexus_widowx_gazebo/meshes/biceps_link.stl" />
+            </geometry>
+            <xacro:material_black />
+         </visual>
+         <collision>
+            <origin xyz="0 0 0" rpy="0 0 0" />
+            <geometry>
+               <mesh filename="package://nexus_widowx_gazebo/meshes/biceps_link.stl" />
             </geometry>
          </collision>
@@ -83,5 +83,5 @@
 			<!--origin xyz="0 0 0" rpy="0 0 0" /-->
             <geometry>
-               <mesh filename="package://nexus_robot/meshes/forearm_link.stl"/>
+               <mesh filename="package://nexus_widowx_gazebo/meshes/forearm_link.stl"/>
             </geometry>
            <xacro:material_black />
@@ -90,5 +90,5 @@
             <origin xyz="0 0 0" rpy="0 0 0" />
             <geometry>
-               <mesh filename="package://nexus_robot/meshes/forearm_link.stl"/>
+               <mesh filename="package://nexus_widowx_gazebo/meshes/forearm_link.stl"/>
             </geometry>
          </collision>
@@ -103,12 +103,12 @@
             <origin xyz="0 0 0" rpy="0 0 0" />
             <geometry>
-               <mesh filename="package://nexus_robot/meshes/wrist_1_link.stl"/>
-            </geometry>
-            <xacro:material_black />
-         </visual>
-         <collision>
-            <origin xyz="0 0 0" rpy="0 0 0" />
-            <geometry>
-               <mesh filename="package://nexus_robot/meshes/wrist_1_link.stl"/>
+               <mesh filename="package://nexus_widowx_gazebo/meshes/wrist_1_link.stl"/>
+            </geometry>
+            <xacro:material_black />
+         </visual>
+         <collision>
+            <origin xyz="0 0 0" rpy="0 0 0" />
+            <geometry>
+               <mesh filename="package://nexus_widowx_gazebo/meshes/wrist_1_link.stl"/>
             </geometry>
          </collision>
@@ -123,12 +123,12 @@
             <origin xyz="0 0 ${M_SCALE*43}" rpy="0 0 0" />
             <geometry>
-               <mesh filename="package://nexus_robot/meshes/wrist_2_link.stl"/>
-            </geometry>
-            <xacro:material_black />
-         </visual>
-         <collision>
-            <origin xyz="0 0 0" rpy="0 0 0" />
-            <geometry>
-               <mesh filename="package://nexus_robot/meshes/wrist_2_link.stl"/>
+               <mesh filename="package://nexus_widowx_gazebo/meshes/wrist_2_link.stl"/>
+            </geometry>
+            <xacro:material_black />
+         </visual>
+         <collision>
+            <origin xyz="0 0 0" rpy="0 0 0" />
+            <geometry>
+               <mesh filename="package://nexus_widowx_gazebo/meshes/wrist_2_link.stl"/>
             </geometry>
          </collision>
@@ -143,12 +143,12 @@
             <origin xyz="0 0 0" rpy="0 0 1.57" />
             <geometry>
-               <mesh filename="package://nexus_robot/meshes/gripper_rail_link.stl"/>
-            </geometry>
-            <xacro:material_black />
-         </visual>
-         <collision>
-            <origin xyz="0 0 0" rpy="0 0 0" />
-            <geometry>
-               <mesh filename="package://nexus_robot/meshes/gripper_rail_link.stl"/>
+               <mesh filename="package://nexus_widowx_gazebo/meshes/gripper_rail_link.stl"/>
+            </geometry>
+            <xacro:material_black />
+         </visual>
+         <collision>
+            <origin xyz="0 0 0" rpy="0 0 0" />
+            <geometry>
+               <mesh filename="package://nexus_widowx_gazebo/meshes/gripper_rail_link.stl"/>
             </geometry>
          </collision>
@@ -165,12 +165,12 @@
             <origin xyz="0 -0.0007 0" rpy="0 0 1.57" />
             <geometry>
-               <mesh filename="package://nexus_robot/meshes/gripper_hand_fixed_link.stl"/>
-            </geometry>
-            <xacro:material_black />
-         </visual>
-         <collision>
-            <origin xyz="0 0 0" rpy="0 0 0" />
-            <geometry>
-               <mesh filename="package://nexus_robot/meshes/gripper_hand_fixed_link.stl"/>
+               <mesh filename="package://nexus_widowx_gazebo/meshes/gripper_hand_fixed_link.stl"/>
+            </geometry>
+            <xacro:material_black />
+         </visual>
+         <collision>
+            <origin xyz="0 0 0" rpy="0 0 0" />
+            <geometry>
+               <mesh filename="package://nexus_widowx_gazebo/meshes/gripper_hand_fixed_link.stl"/>
             </geometry>
          </collision>
@@ -185,12 +185,12 @@
             <origin xyz="0 0.0007 0" rpy="0 0 -1.57" />
             <geometry>
-               <mesh filename="package://nexus_robot/meshes/gripper_hand_fixed_link.stl"/>
-            </geometry>
-            <xacro:material_black />
-         </visual>
-         <collision>
-            <origin xyz="0 0 0" rpy="0 0 0" />
-            <geometry>
-               <mesh filename="package://nexus_robot/meshes/gripper_hand_fixed_link.stl"/>
+               <mesh filename="package://nexus_widowx_gazebo/meshes/gripper_hand_fixed_link.stl"/>
+            </geometry>
+            <xacro:material_black />
+         </visual>
+         <collision>
+            <origin xyz="0 0 0" rpy="0 0 0" />
+            <geometry>
+               <mesh filename="package://nexus_widowx_gazebo/meshes/gripper_hand_fixed_link.stl"/>
             </geometry>
          </collision>
